File: PCB/mostek-h.brd (EAGLE design)
At the start: 97 x 50 mm, 46 parts, among them IC1 MC33932, IC2 REG1117, X2 52745-1490

Commit message: Ready schema
Parts:
- removed AKU, CHAR: (no value), pinhead:1X02/90
- removed C10, C11, C2, C6: (no value), rcl:C0805
- removed C12, C13: (no value), rcl:C1210
- removed C14, C16, C4: (no value), rcl:C0603
- removed C15: (no value), rcl:C1210K
- removed D2, D4, D6: (no value), standardparts:0805.LED
- removed IC1: MC33932, freescale:HSOP44
- removed IC2: REG1117, burr-brown:SOT223
- removed ON/OF: (no value), pinhead:1X03/90
- removed R10, R12, R13, R14, R4, R5, R6, R8, R9: 10k, rcl:R0603
- removed R11, R7: (no value), rcl:R0603
- removed U$2: PAD_SMD_6X1, _zlacza:SMD_6X1
- removed U$3: ST1S14, _układy:HSOP8
- removed U$5, U$6: 1X3.MMT.SH, headers(2mm)(samtec):1X3_MMT.103.01.X.SH
- removed X2: 52745-1490, con-molex:52745-1490
- added EN1, VIN, VOUT: (no value), pinhead:1X02
- added EN2: (no value), pinhead:1X03
- C3: value (none) -> 100uF
- C7: value (none) -> 100nF
- C9: value (none) -> 1nF
- D1: value MBRS130LT3 -> STPS3L60U
- L1: value COIL8.5 -> 8.5uH
- R3: value (none) -> 4.7k
- U$1: value PAD_SMD_6X1 -> ST1S14; device _zlacza:SMD_6X1 -> _układy:HSOP8
- moved U$1 30.9 mm to (6.43, 44.8), flipped to the top, turned to 90 degrees
- renumbered U$4 to L1
Connections:
- removed net +3V3: C11.1, C13.1, IC2.2, R10.1, R14.1, R4.1, R8.1, R9.1, U$1.3, U$2.3, U$5.1, U$6.1
- removed net 5V: C12.1, C2.1, C3.1, C7.1, C9.1, IC2.3, L1.2, R1.1, R13.1, R3.1, U$5.2, U$6.2
- removed net IN11: IC1.43, X2.6
- removed net IN12: IC1.42, X2.5
- removed net IN21: IC1.21, X2.10
- removed net IN22: IC1.20, X2.9
- removed net M1_1: IC1.7, IC1.8, IC1.9, U$1.6
- removed net M1_2: IC1.36, IC1.37, IC1.38, U$1.5
- removed net M1_CSENSE: C4.1, IC1.2, R7.2, X2.8
- removed net M1_EA: U$1.1, X2.12
- removed net M1_EB: U$1.2, X2.11
- removed net M1_PWM: IC1.1, X2.7
- removed net M2_1: IC1.14, IC1.15, IC1.16, U$2.5
- removed net M2_2: IC1.29, IC1.30, IC1.31, U$2.6
- removed net M2_CSENSE: C14.1, IC1.24, R11.2, X2.3
- removed net M2_EA: U$2.1, X2.2
- removed net M2_EB: U$2.2, X2.1
- removed net M2_PWM: IC1.23, X2.4
- removed net N$11: IC1.22, R8.2
- removed net N$12: IC1.25, R10.2
- removed net N$13: IC1.44, R9.2
- removed net N$17: D2.P$2, R12.2
- removed net N$19: D4.P$2, R13.2
- removed net N$20: D6.P$2, R14.2
- removed net N$4: C8.1, U$3.1
- removed net N$6: R3.2, U$3.2
- removed net N$8: IC1.3, R4.2
- removed net N$9: C6.2, IC1.19
- removed net VBAT: C1.1, C10.2, C15.1, C16.1, C5.1, C6.1, IC1.17, IC1.18, IC1.26, IC1.27, IC1.28, IC1.39, IC1.4, IC1.40, IC1.5, IC1.6, ON/OF.1, R12.1, R6.2, U$3.5, U$3.7
- removed net VBAT_MES: R5.2, R6.1, X2.14
- new net EN1: EN1.2, U$1.3
- new net EN2: EN2.2, U$1.5
- new net VIN: EN2.3
- new net VOUT: C3.1, C7.1, C9.1, L1.2, R1.1, R3.1, VOUT.1
- net GND: now also EN1.1, EN2.1, U$1.6, U$1.EXP, VOUT.2; no longer AKU.1, C11.2, C12.2, C13.2, C14.2, C15.2, C16.2, C2.2, C4.2, CHAR.1, D2.P$1, D4.P$1, D6.P$1, IC1.10, IC1.11, IC1.12, IC1.13, IC1.32, IC1.33, IC1.34, IC1.35, IC1.EH@1, IC1.EH@2, IC1.EH@3, IC2.1, R11.1, R5.1, R7.1, U$1.4, U$2.4, U$3.3, U$3.6, U$3.EXP, U$5.3, U$6.3, X2.13
- net N$1: now also C8.1, U$1.1; no longer AKU.2, ON/OF.2
- net N$2: now also C9.2, R1.2, R2.2, U$1.4; no longer CHAR.2, ON/OF.3
- net N$3: now also C8.2, D1.C, L1.1, U$1.8; no longer C10.1, IC1.41
- net N$5: now also C1.1, C5.1, U$1.7, VIN.2; no longer C8.2, D1.C, L1.1, U$3.8
- net N$7: now also R3.2, U$1.2; no longer C9.2, R1.2, R2.2, U$3.4
Routing:
- net VBAT: track 218.2 -> 0.00 mm, vias 4 -> 0
- net +3V3: track 204.7 -> 0.00 mm, vias 11 -> 0
- net 5V: track 165.0 -> 0.00 mm, vias 4 -> 0
- net IN21: track 79.3 -> 0.00 mm, vias 2 -> 0
- net IN22: track 76.2 -> 0.00 mm, vias 2 -> 0
- net M1_EA: track 71.8 -> 0.00 mm, vias 1 -> 0
- net M1_EB: track 70.0 -> 0.00 mm, vias 1 -> 0
- net M1_2: track 69.6 -> 0.00 mm, vias 4 -> 0
- net N$2: track 64.9 -> 0.00 mm
- net GND: track 64.9 -> 0.00 mm, vias 252 -> 0
- net M2_1: track 64.3 -> 0.00 mm, vias 4 -> 0
- net VBAT_MES: track 57.7 -> 0.00 mm
- net M1_CSENSE: track 51.3 -> 0.00 mm
- net M1_PWM: track 41.4 -> 0.00 mm
- net N$5: track 41.3 -> 0.00 mm
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- removed copper zone on layer 1, net GND
- removed copper zone on layer 16, net GND
- removed copper zone on layer 1, net N$10
- removed copper zone on layer 1, net N$14
