File: PCB/mostek-h.sch (EAGLE design)
At the start: 46 parts, among them IC1 MC33932, IC2 REG1117, X2 52745-1490

Commit message: Ready schema
Parts:
- removed AKU, CHAR: (no value), pinhead:PINHD-1X2/90
- removed C10, C11, C2, C6: (no value), rcl:C-EUC0805
- removed C12, C13: (no value), rcl:C-EUC1210
- removed C14, C16, C4: (no value), rcl:C-EUC0603
- removed C15: (no value), rcl:C-EUC1210K
- removed D2, D4, D6: (no value), standardparts:LED.0805
- removed IC1: MC33932, freescale:MC33932
- removed IC2: REG1117, burr-brown:REG1117
- removed ON/OF: (no value), pinhead:PINHD-1X3/90
- removed R10, R12, R13, R14, R4, R5, R6, R8, R9: 10k, rcl:R-EU_R0603
- removed R11, R7: (no value), rcl:R-EU_R0603
- removed U$2: PAD_SMD_6X1, _zlacza:PAD_SMD_6X1
- removed U$3: ST1S14, _układy:ST1S14
- removed U$4: COIL8.5, _elementy:COIL8.5
- removed U$5, U$6: 1X3.MMT.SH, headers(2mm)(samtec):1X3.MMT.SH
- removed X2: 52745-1490, con-molex:52745-1490
- added EN1, VIN, VOUT: (no value), pinhead:PINHD-1X2
- added EN2: (no value), pinhead:PINHD-1X3
- added L1: 8.5uH, _elementy:COIL8.5
- C3: value (none) -> 100uF
- C7: value (none) -> 100nF
- C9: value (none) -> 1nF
- D1: value MBRS130LT3 -> STPS3L60U; SPICEPREFIX (none) -> D
- R3: value (none) -> 4.7k
- U$1: value PAD_SMD_6X1 -> ST1S14; device _zlacza:PAD_SMD_6X1 -> _układy:ST1S14
Connections:
- removed net +3V3: C11.1, C13.1, IC2.VOUT, R10.1, R14.1, R4.1, R8.1, R9.1, U$1.3, U$2.3, U$5.1, U$6.1
- removed net 5V: C12.1, C2.1, C3.1, C7.1, C9.1, IC2.VIN, R1.1, R13.1, R3.1, U$4.2, U$5.2, U$6.2
- removed net IN11: IC1.IN1, X2-6.S
- removed net IN12: IC1.IN2, X2-5.S
- removed net IN21: IC1.IN3, X2-10.S
- removed net IN22: IC1.IN4, X2-9.S
- removed net M1_1: IC1.OUT1, IC1.OUT1@1, IC1.OUT1@2, U$1.6
- removed net M1_2: IC1.OUT2, IC1.OUT2@1, IC1.OUT2@2, U$1.5
- removed net M1_CSENSE: C4.1, IC1.FBA, R7.2, X2-8.S
- removed net M1_EA: U$1.1, X2-12.S
- removed net M1_EB: U$1.2, X2-11.S
- removed net M1_PWM: IC1.D1, X2-7.S
- removed net M2_1: IC1.OUT4, IC1.OUT4@1, IC1.OUT4@2, U$2.5
- removed net M2_2: IC1.OUT3, IC1.OUT3@1, IC1.OUT3@2, U$2.6
- removed net M2_CSENSE: C14.1, IC1.FBB, R11.2, X2-3.S
- removed net M2_EA: U$2.1, X2-2.S
- removed net M2_EB: U$2.2, X2-1.S
- removed net M2_PWM: IC1.D3, X2-4.S
- removed net N$11: IC1.!SFB, R8.2
- removed net N$12: IC1.EN/!D4, R10.2
- removed net N$13: IC1.!SFA, R9.2
- removed net N$17: D2.2, R12.2
- removed net N$19: D4.2, R13.2
- removed net N$20: D6.2, R14.2
- removed net N$4: C8.1, U$3.1
- removed net N$6: R3.2, U$3.2
- removed net N$8: IC1.EN/!D2, R4.2
- removed net N$9: C6.2, IC1.CCPB
- removed net VBAT: C1.1, C10.2, C15.1, C16.1, C5.1, C6.1, IC1.VPWRA, IC1.VPWRA@1, IC1.VPWRA@2, IC1.VPWRA@3, IC1.VPWRA@4, IC1.VPWRB, IC1.VPWRB@1, IC1.VPWRB@2, IC1.VPWRB@3, IC1.VPWRB@4, ON/OF.1, R12.1, R6.2, U$3.5, U$3.7
- removed net VBAT_MES: R5.2, R6.1, X2-14.S
- new net EN1: EN1.2, U$1.EN1
- new net EN2: EN2.2, U$1.EN2
- new net VIN: EN2.3
- new net VOUT: C3.1, C7.1, C9.1, L1.2, R1.1, R3.1, VOUT.1
- net GND: now also EN1.1, EN2.1, U$1.EXP, U$1.GND, VOUT.2; no longer AKU.1, C11.2, C12.2, C13.2, C14.2, C15.2, C16.2, C2.2, C4.2, CHAR.1, D2.1, D4.1, D6.1, IC1.EH@1, IC1.EH@2, IC1.EH@3, IC1.PGNDA, IC1.PGNDA@1, IC1.PGNDA@2, IC1.PGNDA@3, IC1.PGNDB, IC1.PGNDB@1, IC1.PGNDB@2, IC1.PGNDB@3, IC2.GND, R11.1, R5.1, R7.1, U$1.4, U$2.4, U$3.3, U$3.6, U$3.EXP, U$5.3, U$6.3, X2-13.S
- net N$1: now also C8.1, U$1.BOOT; no longer AKU.2, ON/OF.2
- net N$2: now also C9.2, R1.2, R2.2, U$1.FB; no longer CHAR.2, ON/OF.3
- net N$3: now also C8.2, D1.C, L1.1, U$1.SW; no longer C10.1, IC1.CCPA
- net N$5: now also C1.1, C5.1, U$1.VIN, VIN.2; no longer C8.2, D1.C, U$3.8, U$4.1
- net N$7: now also R3.2, U$1.PG; no longer C9.2, R1.2, R2.2, U$3.4
Other:
- note added: "ST1S14 step-down"
- moved on the sheet: C1, C3, C5, C7, C8, C9, D1, R1, R2, R3
