File: PCB/ST1S14.sch (EAGLE design)
At the start: 16 parts

Commit message: Add net name VIN
Connections:
- removed net N$5: C1.1, C5.1, U$1.VIN, VIN.2
- net VIN: now also C1.1, C5.1, U$1.VIN, VIN.2
Changed lines of the file:
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@@
-</segment>
-</net>
-<net name="N$5" class="0">
-<segment>
-<pinref part="U$1" gate="G$1" pin="VIN"/>
-<wire x1="-167.64" y1="320.04" x2="-160.02" y2="320.04" width="0.1524" layer="91"/>
-<wire x1="-160.02" y1="320.04" x2="-160.02" y2="340.36" width="0.1524" layer="91"/>
-<wire x1="-160.02" y1="340.36" x2="-200.66" y2="340.36" width="0.1524" layer="91"/>
-<wire x1="-200.66" y1="340.36" x2="-200.66" y2="322.58" width="0.1524" layer="91"/>
-<wire x1="-200.66" y1="322.58" x2="-228.6" y2="322.58" width="0.1524" layer="91"/>
-<pinref part="C1" gate="G$1" pin="1"/>
-<wire x1="-228.6" y1="322.58" x2="-238.76" y2="322.58" width="0.1524" layer="91"/>
-<wire x1="-228.6" y1="307.34" x2="-228.6" y2="322.58" width="0.1524" layer="91"/>
-<junction x="-228.6" y="322.58"/>
-<wire x1="-238.76" y1="307.34" x2="-238.76" y2="322.58" width="0.1524" layer="91"/>
-<pinref part="C5" gate="G$1" pin="1"/>
-<pinref part="VIN" gate="G$1" pin="2"/>
-<wire x1="-246.38" y1="330.2" x2="-246.38" y2="322.58" width="0.1524" layer="91"/>
-<wire x1="-246.38" y1="322.58" x2="-238.76" y2="322.58" width="0.1524" layer="91"/>
 </segment>
 </net>
@@
 <label x="-218.44" y="342.9" size="1.778" layer="95" rot="R90"/>
 </segment>
+<segment>
+<pinref part="U$1" gate="G$1" pin="VIN"/>
+<wire x1="-167.64" y1="320.04" x2="-160.02" y2="320.04" width="0.1524" layer="91"/>
+<wire x1="-160.02" y1="320.04" x2="-160.02" y2="340.36" width="0.1524" layer="91"/>
+<wire x1="-160.02" y1="340.36" x2="-200.66" y2="340.36" width="0.1524" layer="91"/>
+<wire x1="-200.66" y1="340.36" x2="-200.66" y2="322.58" width="0.1524" layer="91"/>
+<wire x1="-200.66" y1="322.58" x2="-228.6" y2="322.58" width="0.1524" layer="91"/>
+<pinref part="C1" gate="G$1" pin="1"/>
+<wire x1="-228.6" y1="322.58" x2="-238.76" y2="322.58" width="0.1524" layer="91"/>
+<wire x1="-228.6" y1="307.34" x2="-228.6" y2="322.58" width="0.1524" layer="91"/>
+<junction x="-228.6" y="322.58"/>
+<wire x1="-238.76" y1="307.34" x2="-238.76" y2="322.58" width="0.1524" layer="91"/>
+<pinref part="C5" gate="G$1" pin="1"/>
+<pinref part="VIN" gate="G$1" pin="2"/>
+<wire x1="-246.38" y1="330.2" x2="-246.38" y2="322.58" width="0.1524" layer="91"/>
+<wire x1="-246.38" y1="322.58" x2="-238.76" y2="322.58" width="0.1524" layer="91"/>
+</segment>
 </net>

Commit message: Add schema and board comp image
Parts:
- C1: value 100nF -> 10uF
- C5: value 10uF -> 100nF
Connections:
- net GND: now also VIN.1
Changed lines of the file:
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@@
 <attribute name="SPICEPREFIX" value="D"/>
 </part>
-<part name="C1" library="rcl" library_urn="urn:adsk.eagle:library:334" deviceset="C-EU" device="C1210K" package3d_urn="urn:adsk.eagle:package:23683/2" value="100nF"/>
+<part name="C1" library="rcl" library_urn="urn:adsk.eagle:library:334" deviceset="C-EU" device="C1210K" package3d_urn="urn:adsk.eagle:package:23683/2" value="10uF"/>
 <part name="C3" library="rcl" library_urn="urn:adsk.eagle:library:334" deviceset="C-EU" device="C1210K" package3d_urn="urn:adsk.eagle:package:23683/2" value="100uF"/>
-<part name="C5" library="rcl" library_urn="urn:adsk.eagle:library:334" deviceset="C-EU" device="C0603" package3d_urn="urn:adsk.eagle:package:23616/2" value="10uF"/>
+<part name="C5" library="rcl" library_urn="urn:adsk.eagle:library:334" deviceset="C-EU" device="C0603" package3d_urn="urn:adsk.eagle:package:23616/2" value="100nF"/>
 <part name="C7" library="rcl" library_urn="urn:adsk.eagle:library:334" deviceset="C-EU" device="C0603" package3d_urn="urn:adsk.eagle:package:23616/2" value="100nF"/>
 <part name="C8" library="rcl" library_urn="urn:adsk.eagle:library:334" deviceset="C-EU" device="C0603" package3d_urn="urn:adsk.eagle:package:23616/2" value="100nF"/>
@@
 <pinref part="GND14" gate="1" pin="GND"/>
 <wire x1="-248.92" y1="330.2" x2="-248.92" y2="292.1" width="0.1524" layer="91"/>
+<pinref part="VIN" gate="G$1" pin="1"/>
 </segment>
 <segment>
